File: LIC_V-00237-02.brd (EAGLE design)
At the start: 50.5 x 47 mm, 17 parts, among them J1 S4B-PH-SM4-TB

Commit message: Uprava další verze
Další verze s chybou ohledně termálních plošek
Parts:
- R1, R2: value (none) -> 22R0
- R3: value (none) -> 2k2
- moved J1 0.50 mm to (0.20, 22.5)
Routing:
- net 1-: track 81.6 -> 82.6 mm
- net 2-: track 14.1 -> 13.5 mm
Other:
- board size 50.5 x 47 mm -> 48.5 x 45 mm
Changed lines of the file:
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@@
 <layer number="38" name="bTest" color="7" fill="1" visible="no" active="yes"/>
 <layer number="39" name="tKeepout" color="4" fill="11" visible="no" active="yes"/>
-<layer number="40" name="bKeepout" color="1" fill="11" visible="no" active="yes"/>
+<layer number="40" name="bKeepout" color="1" fill="11" visible="yes" active="yes"/>
 <layer number="41" name="tRestrict" color="4" fill="10" visible="no" active="yes"/>
-<layer number="42" name="bRestrict" color="1" fill="10" visible="no" active="yes"/>
+<layer number="42" name="bRestrict" color="1" fill="10" visible="yes" active="yes"/>
 <layer number="43" name="vRestrict" color="2" fill="10" visible="no" active="yes"/>
 <layer number="44" name="Drills" color="7" fill="1" visible="no" active="yes"/>
@@
 <circle x="7" y="3.5" radius="3" width="0.5" layer="21"/>
 <circle x="45" y="3.5" radius="3" width="0.5" layer="21"/>
-<circle x="26" y="22.5" radius="15.5" width="2" layer="46"/>
-<wire x1="47" y1="46" x2="2.5" y2="46" width="2" layer="46"/>
-<wire x1="2.5" y1="46" x2="2.5" y2="32.5" width="2" layer="46"/>
-<wire x1="2.5" y1="32.5" x2="1.5" y2="31.5" width="2" layer="46" curve="-90"/>
-<wire x1="-1" y1="31.5" x2="-1" y2="13.5" width="2" layer="46"/>
-<wire x1="2.5" y1="-1" x2="47" y2="-1" width="2" layer="46"/>
-<wire x1="49.5" y1="1.5" x2="49.5" y2="43.5" width="2" layer="46"/>
-<wire x1="-1" y1="31.5" x2="1.5" y2="31.5" width="2" layer="46"/>
-<wire x1="2.5" y1="-1" x2="2.5" y2="12.5" width="2" layer="46"/>
-<wire x1="-1" y1="13.5" x2="1.5" y2="13.5" width="2" layer="46"/>
-<wire x1="1.5" y1="13.5" x2="2.5" y2="12.5" width="2" layer="46" curve="-90"/>
-<wire x1="47" y1="-1" x2="49.5" y2="1.5" width="2" layer="46"/>
-<wire x1="47" y1="46" x2="49.5" y2="43.5" width="2" layer="46"/>
+<wire x1="17.3" y1="45.3" x2="19.3" y2="41.8" width="0.4064" layer="42"/>
+<wire x1="13.2" y1="39.6" x2="9.9" y2="44.8" width="0.4064" layer="42"/>
+<wire x1="47.6" y1="15.2" x2="48.5" y2="15.2" width="0.4064" layer="42"/>
+<wire x1="46" y1="26.8" x2="48.8" y2="27.5" width="0.4064" layer="42"/>
+<wire x1="46.9" y1="34.6" x2="48.6" y2="34.6" width="0.4064" layer="42"/>
+<wire x1="36.3" y1="40.4" x2="37.6" y2="45" width="0.4064" layer="42"/>
+<wire x1="27.7" y1="43.2" x2="27.8" y2="45.1" width="0.4064" layer="42"/>
+<wire x1="19.7" y1="39.9" x2="20.1" y2="39" width="0.4064" layer="42"/>
+<wire x1="35.2" y1="38.8" x2="34.5" y2="37.8" width="0.4064" layer="42"/>
+<wire x1="42" y1="10.1" x2="44.9" y2="8.3" width="0.4064" layer="42"/>
+<wire x1="35.7" y1="4.7" x2="38.2" y2="1.7" width="0.4064" layer="42"/>
+<wire x1="33.8" y1="7.9" x2="34.9" y2="6.5" width="0.4064" layer="42"/>
+<wire x1="39" y1="12.8" x2="40.8" y2="11.7" width="0.4064" layer="42"/>
+<wire x1="27.7" y1="5.9" x2="28" y2="4.3" width="0.4064" layer="42"/>
+<wire x1="28.4" y1="2.3" x2="28.6" y2="1" width="0.4064" layer="42"/>
+<wire x1="19.9" y1="5" x2="20.6" y2="6.8" width="0.4064" layer="42"/>
+<wire x1="13.7" y1="8.9" x2="14.9" y2="10.2" width="0.4064" layer="42"/>
+<wire x1="10.6" y1="6.4" x2="12.1" y2="7.6" width="0.4064" layer="42"/>
 </plain>
 <attributes>
@@
 </class>
 </classes>
-<designrules name="Michal_small *">
+<designrules name="Michal_small">
 <description language="cs">&lt;b&gt;Mucha návrh - small&lt;/b&gt;
 &lt;p&gt;
@@
 <element name="D8" library="led" package="OSRAM_LCW" value="OSRAM_LCW_CQ7P.EC-KTLP-5J7K-1-K" x="16.3" y="39.4" rot="MR150"/>
 <element name="D9" library="led" package="OSRAM_LCW" value="OSRAM_LCW_CQ7P.EC-KTLP-5J7K-1-K" x="24" y="42" rot="MR180"/>
-<element name="J1" library="con-jst" package="S4B-PH-SM4-TB" value="S4B-PH-SM4-TB" x="0.2" y="22" rot="MR270"/>
-<element name="R1" library="rcl" package="R1206" value="" x="44.5" y="35.5" rot="MR0"/>
-<element name="R3" library="rcl" package="R1206" value="" x="5.5" y="32.5" rot="MR270"/>
-<element name="R2" library="rcl" package="R1206" value="" x="13.5" y="37" rot="MR45"/>
+<element name="J1" library="con-jst" package="S4B-PH-SM4-TB" value="S4B-PH-SM4-TB" x="0.2" y="22.5" rot="MR270"/>
+<element name="R1" library="rcl" package="R1206" value="22R0" x="44.5" y="35.5" rot="MR0"/>
+<element name="R3" library="rcl" package="R1206" value="2k2" x="5.5" y="32.5" rot="MR270"/>
+<element name="R2" library="rcl" package="R1206" value="22R0" x="13.5" y="37" rot="MR45"/>
 </elements>
 <signals>
@@
 <contactref element="D11" pad="THERMAL"/>
 <contactref element="D12" pad="THERMAL"/>
-<polygon width="0.4064" layer="16" thermals="no" rank="3">
+<polygon width="0.4064" layer="16" isolate="0.3048" thermals="no" rank="3">
 <vertex x="0" y="0"/>
 <vertex x="49.5" y="0"/>
@@
 <contactref element="J1" pad="GND1"/>
 <contactref element="J1" pad="GND2"/>
+<wire x1="24" y1="3.1" x2="16.3" y2="5.6" width="0" layer="19" extent="16-16"/>
+<wire x1="32" y1="4" x2="24" y2="3.1" width="0" layer="19" extent="16-16"/>
+<wire x1="39" y1="8" x2="32" y2="4" width="0" layer="19" extent="16-16"/>
+<wire x1="10.2" y1="11" x2="16.3" y2="5.6" width="0" layer="19" extent="16-16"/>
+<wire x1="43.8" y1="14.6" x2="39" y2="8" width="0" layer="19" extent="16-16"/>
 <wire x1="45.5" y1="22.5" x2="43.8" y2="14.6" width="0" layer="19" extent="16-16"/>
+<wire x1="43.8" y1="30.4" x2="45.5" y2="22.5" width="0" layer="19" extent="16-16"/>
+<wire x1="39" y1="37" x2="43.8" y2="30.4" width="0" layer="19" extent="16-16"/>
+<wire x1="32" y1="41" x2="39" y2="37" width="0" layer="19" extent="16-16"/>
+<wire x1="24" y1="42" x2="32" y2="41" width="0" layer="19" extent="16-16"/>
+<wire x1="16.3" y1="39.4" x2="24" y2="42" width="0" layer="19" extent="16-16"/>
+<wire x1="10.2" y1="34" x2="16.3" y2="39.4" width="0" layer="19" extent="16-16"/>
 </signal>
 <signal name="N$1">
@@
 <contactref element="J1" pad="3"/>
 <contactref element="D7" pad="C"/>
-<wire x1="8.45" y1="23" x2="5.5" y2="23" width="0.4064" layer="16"/>
-<wire x1="5.5" y1="23" x2="5.6" y2="25.9" width="0.4064" layer="16"/>
+<wire x1="8.45" y1="23.5" x2="5.6" y2="23.5" width="0.4064" layer="16"/>
+<wire x1="5.6" y1="23.5" x2="5.6" y2="25.9" width="0.4064" layer="16"/>
 <wire x1="5.6" y1="25.9" x2="7" y2="27.5" width="0.4064" layer="16"/>
 <wire x1="7" y1="27.5" x2="9.53874375" y2="33.089853125" width="0.4064" layer="16"/>
@@
 <contactref element="J1" pad="1"/>
 <wire x1="9.3" y1="12.2" x2="8.45" y2="13.05" width="1" layer="16"/>
-<wire x1="8.45" y1="13.05" x2="8.45" y2="19" width="1" layer="16"/>
+<wire x1="8.45" y1="13.05" x2="8.45" y2="19.5" width="1" layer="16"/>
 <contactref element="D6" pad="C"/>
 <contactref element="D13" pad="C"/>
@@
 <wire x1="5.5" y1="10.5" x2="5.5" y2="14.5" width="0.4064" layer="16"/>
 <wire x1="5.5" y1="14.5" x2="4.5" y2="15.5" width="0.4064" layer="16"/>
-<wire x1="4.5" y1="15.5" x2="4.5" y2="18.5" width="0.4064" layer="16"/>
-<wire x1="4.5" y1="18.5" x2="5" y2="19" width="0.4064" layer="16"/>
-<wire x1="5" y1="19" x2="8.45" y2="19" width="0.4064" layer="16"/>
+<wire x1="4.5" y1="15.5" x2="4.5" y2="19" width="0.4064" layer="16"/>
+<wire x1="4.5" y1="19" x2="5" y2="19.5" width="0.4064" layer="16"/>
+<wire x1="5" y1="19.5" x2="8.45" y2="19.5" width="0.4064" layer="16"/>
 <wire x1="47" y1="17" x2="45.5" y2="21.375" width="0.4064" layer="16" curve="37.849284"/>
 <wire x1="9.3" y1="12.2" x2="9.53874375" y2="11.91014375" width="0.4064" layer="16" curve="-11.045986"/>
@@
 <contactref element="R3" pad="2"/>
 <contactref element="J1" pad="2"/>
-<wire x1="8.45" y1="21" x2="4.5" y2="21" width="0.4064" layer="16"/>
-<wire x1="4.5" y1="21" x2="3.5" y2="22.5" width="0.4064" layer="16" curve="-112.619814"/>
-<wire x1="3.5" y1="22.5" x2="4.5" y2="30.5" width="0.4064" layer="16"/>
+<wire x1="8.45" y1="21.5" x2="4.5" y2="21.5" width="0.4064" layer="16"/>
+<wire x1="4.5" y1="21.5" x2="3.5" y2="23" width="0.4064" layer="16" curve="-112.619814"/>
+<wire x1="3.5" y1="23" x2="4.5" y2="30.5" width="0.4064" layer="16"/>
 <wire x1="4.5" y1="30.5" x2="5.5" y2="31.05" width="0.4064" layer="16"/>
 </signal>
@@
 <contactref element="D8" pad="A"/>
 <contactref element="R2" pad="2"/>
-<wire x1="8.45" y1="25" x2="8.5" y2="25.3" width="1.016" layer="16"/>
-<wire x1="8.5" y1="25.3" x2="9" y2="27.4" width="1.016" layer="16" curve="-51.496116"/>
+<wire x1="8.45" y1="25.5" x2="8.5" y2="26.2" width="1.016" layer="16"/>
+<wire x1="8.5" y1="26.2" x2="9" y2="27.4" width="1.016" layer="16" curve="-51.496116"/>
 <wire x1="9" y1="27.4" x2="11" y2="31" width="1.016" layer="16" curve="20.171886"/>
 <wire x1="11" y1="31" x2="12.7" y2="33.5" width="0.4064" layer="16"/>
@@
 <contactref element="D7" pad="A"/>
 <contactref element="R3" pad="1"/>
-<wire x1="10.861259375" y1="34.91014375" x2="9" y2="36" width="0.4064" layer="16"/>
-<wire x1="9" y1="36" x2="5.5" y2="33.95" width="0.4064" layer="16" curve="121.418166"/>
+<wire x1="10.861259375" y1="34.91014375" x2="8.8" y2="36.4" width="0.4064" layer="16"/>
+<wire x1="8.8" y1="36.4" x2="5.5" y2="33.95" width="0.4064" layer="16" curve="121.418166"/>
 </signal>
 <signal name="N$6">

Commit message: Další verze
Verze pro normální LED
Parts:
- removed D1, D10, D11, D12, D13, D2, D3, D4, D5, D6, D8, D9: OSRAM_LCW_CQ7P.EC-KTLP-5J7K-1-K, led:OSRAM_LCW
- removed R3: 2k2, rcl:R1206
- added D14, D15, D16, D17, D18, D19, D20, D21, D22, D23, D24: (no value), #PaJa_31:P1206
- added R5: 0R, rcl:R1206
- D7: value OSRAM_LCW_CQ7P.EC-KTLP-5J7K-1-K -> (none); device led:OSRAM_LCW -> #PaJa_31:P1206
- moved R1 38.7 mm to (6.00, 31.5), turned to 270 degrees
- moved R2 24.7 mm to (6.00, 13.5), turned to 90 degrees
- moved D7 23.0 mm to (10.2, 11.0), turned to 234 degrees
Connections:
- removed net THERMAL: D1.THERMAL, D10.THERMAL, D11.THERMAL, D12.THERMAL, D13.THERMAL, D2.THERMAL, D3.THERMAL, D4.THERMAL, D5.THERMAL, D6.THERMAL, D7.THERMAL, D8.THERMAL, D9.THERMAL, J1.GND1, J1.GND2
- new net GND: J1.GND1, J1.GND2
- net 1+: now also R1.2; no longer D8.A, R2.2
- net 1-: now also R5.2; no longer D13.C, D6.C
- net 2+: now also R2.2; no longer R3.2
- net 2-: now also D18.K; no longer D7.C
- net N$1: now also D14.A, D7.K; no longer D1.C, D2.A
- net N$10: now also D22.K, D23.A; no longer D12.A, R1.1
- net N$11: now also D19.A, R1.1; no longer D11.C, R1.2
- net N$12: now also D24.K, R5.1; no longer D7.A, R3.1
- net N$14: now also D23.K, D24.A; no longer D12.C, D13.A
- net N$2: now also D14.K, D15.A; no longer D2.C, D3.A
- net N$3: now also D15.K, D16.A; no longer D3.C, D4.A
- net N$4: now also D16.K, D17.A; no longer D4.C, D5.A
- net N$5: now also D17.K, D18.A; no longer D5.C, D6.A
- net N$6: now also D7.A; no longer D1.A
- net N$7: now also D19.K, D20.A; no longer D8.C, D9.A
- net N$8: now also D20.K, D21.A; no longer D10.A, D9.C
- net N$9: now also D21.K, D22.A; no longer D10.C, D11.A
Routing:
- net 2-: track 13.5 -> 70.0 mm
- net N$6: track 37.9 -> 3.28 mm
- net 1-: track 82.6 -> 49.3 mm
- net 1+: track 16.6 -> 5.56 mm
- net 2+: track 14.5 -> 8.99 mm
- net N$3: track 6.08 -> 4.61 mm
- net N$9: track 6.04 -> 4.62 mm
- net N$2: track 6.08 -> 4.69 mm
- net N$8: track 6.07 -> 4.72 mm
- net N$4: track 5.95 -> 4.67 mm
- net N$7: track 5.99 -> 4.73 mm
- net N$1: track 5.97 -> 4.73 mm
- net N$5: track 5.97 -> 4.75 mm
- net N$14: track 5.89 -> 4.75 mm
- net N$12: track 6.65 -> 7.49 mm
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- added copper zone on layer 16, net GND
- removed copper zone on layer 16, net THERMAL
Other:
- outline, holes or cut-outs redrawn
